File: Tasmodul_RasPi_LoRa.brd (EAGLE design)
At the start: 100 x 100 mm, 60 parts, among them J1 691322310002, J2 RASPI_4B, J3 LORA_MPCIE, J4 636101111001, J5 60311002111526, J6 60311002111526, Q1 DMN3404L-7, U1 AP64351, U2 QUECTEL_L76-M33, U3 REG1117

Commit message: * Added more description to the schematic * Added more silk screen information to the PCB * Added U.fl connectors for the SMA connectors as a backup
Parts:
- added J7, J8: 60311002111526, Wurth_Connectors_WR-SMA:60311002111526
- C17, C21: value (none) -> dnp
- J5, J6: value 60311002111526 -> 636101111001; device Wurth_Connectors_WR-SMA:60311002111526 -> Wurth_Connectors_WR-UMRF:636101111001
- R10: value (none) -> 10R
- R11: value (none) -> 0R
- moved J5 6.50 mm to (11.5, 86.0), flipped to the bottom, turned to 90 degrees
- moved J6 6.50 mm to (11.5, 70.5), flipped to the bottom, turned to 90 degrees
Connections:
- new net HF_GNSS: J6.1, J8.1
- new net HF_LORA: J5.1, J7.1
- net GND: now also J7.2, J7.3, J7.4, J7.5, J8.2, J8.3, J8.4, J8.5; no longer J5.4, J5.5, J6.4, J6.5
Routing:
- net GND: track 11.1 -> 16.5 mm, vias 160 -> 193
- net HF_LORA: track 0.00 -> 4.97 mm
- net HF_GNSS: track 0.00 -> 4.97 mm
Other:
- outline, holes or cut-outs redrawn
- board text added: "Fan: GPIO17"
- board text added: "mPCIe LoRa Card SPI only!"
- board text removed: "mPCIE LoRa Card"

Commit message: * Added multifuse to power input * Added I2C pullup resistors * Added test points to unused GPS module pins * Updated README.md
Parts:
- added F1: 1812L150, Fuse:FUSC4532X125
- added R12: 10R, rcl:R0603
- added R13, R14: 0R, rcl:R0603
- added TP1, TP2, TP3: TPTP15R, testpad:TP15R
- C10: value (none) -> dnp
- C15, C16, C19, C20, C8: value (none) -> 100n
- C9: value dnp -> 100n
- LED1: value (none) -> green
- Q1: value DMN3404L-7 -> 5.8A/30V/35mΩ
- R10: value 10R -> 22k1
- R11: value 0R -> 1k
- R6: value 15k8 -> 4k7
- R7: value 115k -> 4k7
- R8: value 22k1 -> 15k8
- R9: value (none) -> 115k
- moved R10 55.1 mm to (81.0, 74.0), flipped to the top, turned to 270 degrees
- moved R11 46.8 mm to (76.5, 73.0), flipped to the top
- moved C10 30.4 mm to (77.5, 70.0), flipped to the top
- moved C9 30.4 mm to (48.0, 77.5), flipped to the bottom
- moved R6 18.6 mm to (75.0, 53.5), turned to 270 degrees
- moved R7 16.6 mm to (77.5, 53.5)
- moved D1 7.07 mm to (81.0, 81.0), turned to 180 degrees
- moved R8 4.72 mm to (83.5, 70.0), turned to 90 degrees
- moved R9 4.24 mm to (79.5, 70.0), turned to 270 degrees
- moved B1 0.50 mm to (50.0, 87.5)
Connections:
- new net N$13: J2.1, R6.2, R7.2
- new net N$15: F1.1, J1.2
- new net N$16: TP1.TP, U2.16
- new net N$17: TP2.TP, U2.17
- new net N$18: TP3.TP, U2.18
- new net N$19: J3.25, R14.2
- net +3V3: now also C9.1; no longer C10.1
- net +5V: now also C10.2, R9.2; no longer C9.2, R7.2
- net GND: now also C9.2, R10.1, R11.1; no longer C10.2, R8.1, R9.1
- net GPS_STBY: now also R14.1; no longer J3.25
- net I2C_SCL: now also R6.1
- net I2C_SDA: now also R7.1
- net N$10: now also R12.2; no longer R10.2
- net N$11: now also R8.1; no longer R6.1
- net N$12: now also R8.2; no longer R6.2
- net N$4: now also R12.1; no longer R10.1
- net N$6: now also C10.1, R10.2, R9.1; no longer C9.1, R7.1, R8.2
- net N$7: now also R11.2; no longer R9.2
- net RF_CON: now also R13.1; no longer R11.1
- net RF_MATCHED: now also R13.2; no longer R11.2
- net VIN: now also F1.2; no longer J1.2
Routing:
- net N$13: track 0.00 -> 11.0 mm, vias 0 -> 2
- net N$19: track 0.00 -> 5.90 mm
- net N$15: track 0.00 -> 5.59 mm
- net N$18: track 0.00 -> 5.28 mm
- net N$17: track 0.00 -> 4.35 mm
- net GPS_STBY: track 78.6 -> 82.8 mm
- net N$16: track 0.00 -> 3.98 mm
- net VIN: track 14.4 -> 10.6 mm
- net I2C_SCL: track 35.3 -> 38.1 mm
- net I2C_SDA: track 38.4 -> 41.2 mm
- net GPS_TXD: track 67.2 -> 66.4 mm
- net GPS_RXD: track 60.2 -> 59.4 mm
- net VBAT: track 6.52 -> 7.02 mm
- net GND: vias 193 -> 194

Commit message: * Added 3 status LEDs to the RasPi * Minor Layout tweaks
Parts:
- added LED2, LED3, LED4: green, led:CHIPLED_0603
- added R15: 10R, rcl:R0603
- added R16, R17: 0R, rcl:R0603
- C13: value 100n -> 1u
- C14: value 1u -> dnp
- C17, C21: value dnp -> 100n
- C19: value 100n -> dnp
- R10: value 22k1 -> 4k7
- R11: value 1k -> 4k7
- R12: value 10R -> 115k
- R13: value 0R -> 22k1
- R14, R3: value 0R -> 1k
- R2: value 100R -> 1k
- R4: value nc -> 1k
- R5: value 1k -> 100R
- R6: value 4k7 -> 0R
- R7: value 4k7 -> nc
- R8: value 15k8 -> 1k
- R9: value 115k -> 15k8
- moved R12 54.3 mm to (79.5, 70.0), flipped to the top, turned to 270 degrees
- moved R13 51.2 mm to (81.0, 74.0), flipped to the top, turned to 270 degrees
- moved C14 48.7 mm to (32.5, 79.0), flipped to the bottom
- moved C21 47.8 mm to (74.5, 87.5), flipped to the top
- moved C19 46.3 mm to (27.5, 79.0), flipped to the bottom
- moved R5 44.6 mm to (71.5, 43.5), flipped to the top, turned to 90 degrees
- moved R8 36.5 mm to (49.0, 82.0), flipped to the bottom, turned to 180 degrees
- moved LED1 33.6 mm to (94.0, 42.0), turned to 180 degrees
- moved R4 28.0 mm to (92.0, 54.0), turned to 90 degrees
- moved C17 27.3 mm to (59.5, 83.0), flipped to the top, turned to 90 degrees
- moved C18 25.5 mm to (59.5, 71.0), turned to 90 degrees
- moved R3 24.9 mm to (92.0, 48.0), turned to 90 degrees
- moved C16 22.5 mm to (59.5, 93.5), turned to 270 degrees
- moved C13 21.8 mm to (80.5, 87.5)
- moved R10 21.4 mm to (75.0, 53.5)
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Connections:
- new net N$20: LED1.C, R2.1
- new net N$21: LED2.C, R3.1
- new net N$22: LED3.C, R4.1
- new net N$23: J2.7, LED1.A
- new net N$24: J2.29, LED2.A
- new net N$25: J2.31, LED3.A
- net +3V3: now also C17.1, C18.1, C21.1; no longer C13.1, C15.1, C19.1
- net +5V: now also C13.1, C15.1, LED4.A, R12.2; no longer C14.1, C18.1, LED1.A, R9.2
- net FAN: now also R5.2; no longer R2.2
- net GND: now also C14.1, C17.2, C19.1, C21.2, R13.1, R14.1, R2.2, R3.2, R4.2; no longer C14.2, C17.1, C19.2, C21.1, R10.1, R11.1
- net GPS_STBY: now also R17.1; no longer R14.1
- net I2C_SCL: now also R10.1; no longer R6.1
- net I2C_SDA: now also R11.1; no longer R7.1
- net LORA_RESET: now also R6.2, R7.2; no longer R3.2, R4.2
- net N$1: now also R7.1; no longer R4.1
- net N$10: now also R15.2; no longer R12.2
- net N$11: now also R9.1; no longer R8.1
- net N$12: now also R9.2; no longer R8.2
- net N$13: now also R10.2, R11.2; no longer R6.2, R7.2
- net N$19: now also R17.2; no longer R14.2
- net N$3: now also R6.1; no longer R3.1
- net N$4: now also R15.1; no longer R12.1
- net N$6: now also R12.1, R13.2; no longer R10.2, R9.1
- net N$7: now also LED4.C, R14.2; no longer LED1.C, R11.2
- net N$8: now also R8.2; no longer R5.2
- net N$9: now also R5.1; no longer R2.1
- net RF_CON: now also C19.2, R16.1; no longer C21.2, R13.1
- net RF_MATCHED: now also C14.2, R16.2; no longer C17.2, R13.2
- net VBAT: now also R8.1; no longer R5.1
Routing:
- net N$25: track 0.00 -> 62.8 mm, vias 0 -> 2
- net N$24: track 0.00 -> 55.0 mm, vias 0 -> 2
- net N$23: track 0.00 -> 41.3 mm, vias 0 -> 2
- net GPS_STBY: track 82.8 -> 79.3 mm
- net GPS_TXD: track 66.4 -> 68.5 mm
- net GPS_RXD: track 59.4 -> 61.5 mm
- net N$22: track 0.00 -> 2.04 mm
- net N$21: track 0.00 -> 2.04 mm
- net N$20: track 0.00 -> 2.04 mm
- net N$13: track 11.0 -> 9.43 mm, vias 2 -> 0
- net +5V: track 127.8 -> 128.8 mm
- net LORA_GPS_TXD: track 27.3 -> 28.3 mm
- net LORA_GPS_RXD: track 21.1 -> 22.1 mm
- net SX1302_GPIO6: track 18.3 -> 19.0 mm
- net N$19: track 5.90 -> 5.40 mm
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- added copper zone on layer 16, net +3V3
Other:
- board text added: "5V ok"
- board text added: "U1"
- board text added: "U2"
- board text added: "WAN"
